Commit message: Modified CMakelists.txt and created core URDF

File: description/robot.urdf.xacro (robot description, xacro)
@@ -1,5 +1,4 @@
 <?xml version="1.0"?>
-<robot xmlns:xacro="http://www.ros.org/wiki/xacro"  name="robot">
-    <!-- Example link-->
-    <link name="base_link"></link>
+<robot xmlns:xacro="http://www.ros.org/wiki/xacro"  name="differential_bot">
+    <xacro:include filename="robot_core.xacro"/>
 </robot>

Commit message: Added Gazebo simulation with gazebo differential robot control plugin

File: description/robot.urdf.xacro (robot description, xacro)
@@ -2,3 +2,4 @@
 <robot xmlns:xacro="http://www.ros.org/wiki/xacro"  name="differential_bot">
     <xacro:include filename="robot_core.xacro"/>
+    <xacro:include filename="gazebo_control.xacro"/>
 </robot>

File: description/robot_core.xacro (robot description, xacro)
@@ -41,4 +41,7 @@
         </xacro:inertial_box>
     </link>
+    <gazebo reference="chassis">
+        <material>Gazebo/White</material>
+    </gazebo>
     <!-- LEFT WHEEL LINK-->
      <!-- We could connect the wheels to the chassis, but we will
@@ -67,4 +70,7 @@
         </xacro:inertial_cylinder>
     </link>
+    <gazebo reference="left_wheel">
+        <material>Gazebo/Blue</material>
+    </gazebo>
     <!-- RIGHT WHEEL LINK-->
     <joint name="right_wheel_joint" type="continuous">
@@ -90,4 +96,7 @@
         </xacro:inertial_cylinder>
     </link>
+    <gazebo reference="right_wheel">
+        <material>Gazebo/Blue</material>
+    </gazebo>
     <!-- CASTER WHEEL-->
     <joint name="caster_wheel_joint" type="fixed">
@@ -112,3 +121,8 @@
         </xacro:inertial_sphere>
     </link>
+    <gazebo reference="caster_wheel">
+        <material>Gazebo/Black</material>
+        <mu1 value="0.001"/>
+        <mu2 value="0.001"/>
+    </gazebo>
 </robot>

Commit message: Added lidar sensor.

File: description/robot.urdf.xacro (robot description, xacro)
@@ -3,3 +3,4 @@
     <xacro:include filename="robot_core.xacro"/>
     <xacro:include filename="gazebo_control.xacro"/>
+    <xacro:include filename="lidar.xacro"/>
 </robot>

File: description/robot_colors.xacro (robot description, xacro)
@@ -13,3 +13,6 @@
         <color rgba="0 0 0 1" />
     </material>
+    <material name="red">
+        <color rgba="1 0 0 1" />
+    </material>
 </robot>

Commit message: Added toggle option in launch to switch between ros2_control and gazebo_control

File: description/robot.urdf.xacro (robot description, xacro)
@@ -1,7 +1,13 @@
 <?xml version="1.0"?>
 <robot xmlns:xacro="http://www.ros.org/wiki/xacro"  name="differential_bot">
+    <xacro:arg name="use_ros2_control" default="true"/>
     <xacro:include filename="robot_core.xacro"/>
-    <!-- <xacro:include filename="gazebo_control.xacro"/> -->
-    <xacro:include filename="ros2_control.xacro"/>
+    <!-- Check whether to use the ros2_control plugin or the gazebo_control plugin -->
+    <xacro:if value="$(arg use_ros2_control)">
+        <xacro:include filename="ros2_control.xacro"/>
+    </xacro:if>
+    <xacro:unless value="$(arg use_ros2_control)">
+        <xacro:include filename="gazebo_control.xacro"/>
+    </xacro:unless>
     <xacro:include filename="lidar.xacro"/>
     <xacro:include filename="camera.xacro"/>

File: description/robot_core.xacro (robot description, xacro)
@@ -63,5 +63,5 @@
         <collision>
             <geometry>
-                <cylinder radius="0.05" length="0.04"/>
+                <sphere radius="0.05" />
             </geometry>
         </collision>
@@ -89,5 +89,5 @@
         <collision>
             <geometry>
-                <cylinder radius="0.05" length="0.04"/>
+                <sphere radius="0.05" />
             </geometry>
         </collision>
