Commit message: Added base_footprint link and joint, added slam_toolbox online async parameters, added office world

File: description/robot_core.xacro (robot description, xacro)
@@ -3,5 +3,5 @@
     <xacro:include filename="robot_colors.xacro"/>
     <xacro:include filename="inertial_macros.xacro"/>
-    <!-- BASE LINK-->
+    <!-- BASE LINK -->
     <!-- It wouldn't be wrong to put the base link at the center of our
      chassis. But, since this is a differential robot, it's better to put
@@ -10,4 +10,12 @@
      Also, note that URDF uses meters. -->
     <link name="base_link">
+    </link>
+    <!-- BASE_FOOTPRINT LINK -->
+    <joint name="base_footprint_joint" type="fixed">
+        <parent link="base_link"/>
+        <child link="base_footprint"/>
+        <origin xyz="0 0 0" rpy="0 0 0"/>
+    </joint>
+    <link name="base_footprint">
     </link>
     <!-- CHASSIS LINK-->
