Commit message: Added ball tracking params and launch file and configured twist_mux params to include the /cmd_vel_tracker topic and tweaked camera pitch

File: description/camera.xacro (robot description, xacro)
@@ -4,5 +4,5 @@
         <parent link="chassis"/>
         <child link="camera_link"/>
-        <origin xyz="0.305 0 0.08" rpy="0 0 0"/>
+        <origin xyz="0.305 0 0.08" rpy="0 0.181 0"/>
     </joint>
     <!--
